File: schematic/IoTFanControl/IoTFanControl.kicad_sch (KiCad schematic)
At the start: 17 parts, among them J1 Fan1, J2 Fan2, J3 Jumper

Commit message: wipZ
Parts:
- R1, R2, R3: value (none) -> 92R
- SW1, SW2: value (none) -> SW_SPST
- U1: value (none) -> Pico; footprint (none) -> RPi_Pico:RPi_Pico_SMD_TH
Connections:
- net GND: now also U1.14 (GPIO10); no longer U1.15 (GPIO11)
- net at C?.1, SW?.A: now also U1.15 (GPIO11); no longer U1.16 (GPIO12)
- net at SW?.S1: now also U1.16 (GPIO12)
Changed lines of the file:
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@@
-    (stroke (width 0) (type default) (color 0 0 0 0))
-  )
-  (wire (pts (xy 86.36 92.71) (xy 119.38 92.71))
     (stroke (width 0) (type default) (color 0 0 0 0))
   )
@@
     (stroke (width 0) (type default) (color 0 0 0 0))
   )
+  (wire (pts (xy 90.17 95.25) (xy 90.17 106.68))
+    (stroke (width 0) (type default) (color 0 0 0 0))
+  )
   (wire (pts (xy 57.15 140.97) (xy 92.71 140.97))
     (stroke (width 0) (type default) (color 0 0 0 0))
@@
     (stroke (width 0) (type default) (color 0 0 0 0))
   )
+  (wire (pts (xy 86.36 90.17) (xy 119.38 90.17))
+    (stroke (width 0) (type default) (color 0 0 0 0))
+  )
   (wire (pts (xy 49.53 90.17) (xy 58.42 90.17))
     (stroke (width 0) (type default) (color 0 0 0 0))
@@
     (stroke (width 0) (type default) (color 0 0 0 0))
   )
+  (wire (pts (xy 119.38 95.25) (xy 90.17 95.25))
+    (stroke (width 0) (type default) (color 0 0 0 0))
+  )
+  (wire (pts (xy 86.36 73.66) (xy 86.36 90.17))
+    (stroke (width 0) (type default) (color 0 0 0 0))
+  )
   (wire (pts (xy 80.01 64.77) (xy 80.01 57.15))
     (stroke (width 0) (type default) (color 0 0 0 0))
@@
     (stroke (width 0) (type default) (color 0 0 0 0))
   )
+  (wire (pts (xy 29.21 106.68) (xy 29.21 92.71))
+    (stroke (width 0) (type default) (color 0 0 0 0))
+  )
   (wire (pts (xy 49.53 102.87) (xy 58.42 102.87))
     (stroke (width 0) (type default) (color 0 0 0 0))
   )
-  (wire (pts (xy 86.36 95.25) (xy 119.38 95.25))
-    (stroke (width 0) (type default) (color 0 0 0 0))
-  )
   (wire (pts (xy 58.42 73.66) (xy 43.18 73.66))
     (stroke (width 0) (type default) (color 0 0 0 0))
@@
     (stroke (width 0) (type default) (color 0 0 0 0))
   )
+  (wire (pts (xy 29.21 92.71) (xy 34.29 92.71))
+    (stroke (width 0) (type default) (color 0 0 0 0))
+  )
   (wire (pts (xy 119.38 102.87) (xy 106.68 102.87))
     (stroke (width 0) (type default) (color 0 0 0 0))
@@
     (stroke (width 0) (type default) (color 0 0 0 0))
   )
+  (wire (pts (xy 119.38 92.71) (xy 86.36 92.71))
+    (stroke (width 0) (type default) (color 0 0 0 0))
+  )
   (wire (pts (xy 118.11 140.97) (xy 111.76 140.97))
     (stroke (width 0) (type default) (color 0 0 0 0))
@@
     (stroke (width 0) (type default) (color 0 0 0 0))
   )
-  (wire (pts (xy 86.36 102.87) (xy 86.36 95.25))
+  (wire (pts (xy 86.36 92.71) (xy 86.36 102.87))
     (stroke (width 0) (type default) (color 0 0 0 0))
   )
@@
     (stroke (width 0) (type default) (color 0 0 0 0))
   )
-  (wire (pts (xy 86.36 73.66) (xy 86.36 92.71))
-    (stroke (width 0) (type default) (color 0 0 0 0))
-  )
   (wire (pts (xy 71.12 49.53) (xy 96.52 49.53))
     (stroke (width 0) (type default) (color 0 0 0 0))
@@
     (stroke (width 0) (type default) (color 0 0 0 0))
   )
+  (wire (pts (xy 90.17 106.68) (xy 29.21 106.68))
+    (stroke (width 0) (type default) (color 0 0 0 0))
+  )
   (wire (pts (xy 43.18 73.66) (xy 43.18 82.55))
     (stroke (width 0) (type default) (color 0 0 0 0))
@@
     (in_bom yes) (on_board yes)
     (property "Reference" "U1" (id 0) (at 137.16 50.419 0))
-    (property "Value" "" (id 1) (at 137.16 52.7304 0))
-    (property "Footprint" "" (id 2) (at 137.16 81.28 90)
+    (property "Value" "Pico" (id 1) (at 137.16 52.7304 0))
+    (property "Footprint" "RPi_Pico:RPi_Pico_SMD_TH" (id 2) (at 137.16 81.28 90)
       (effects (font (size 1.27 1.27)) hide)
     )
@@
     (in_bom yes) (on_board yes) (fields_autoplaced)
     (property "Reference" "SW1" (id 0) (at 53.34 46.7192 0))
-    (property "Value" "" (id 1) (at 53.34 49.2561 0))
+    (property "Value" "SW_SPST" (id 1) (at 53.34 49.2561 0))
     (property "Footprint" "" (id 2) (at 53.34 52.07 0)
       (effects (font (size 1.27 1.27)) hide)
@@
     (in_bom yes) (on_board yes) (fields_autoplaced)
     (property "Reference" "R3" (id 0) (at 111.76 67.6742 90))
-    (property "Value" "" (id 1) (at 111.76 70.2111 90))
+    (property "Value" "92R" (id 1) (at 111.76 70.2111 90))
     (property "Footprint" "" (id 2) (at 111.76 74.168 90)
       (effects (font (size 1.27 1.27)) hide)
@@
     (in_bom yes) (on_board yes) (fields_autoplaced)
     (property "Reference" "R1" (id 0) (at 111.76 60.0542 90))
-    (property "Value" "" (id 1) (at 111.76 62.5911 90))
+    (property "Value" "92R" (id 1) (at 111.76 62.5911 90))
     (property "Footprint" "" (id 2) (at 111.76 66.548 90)
       (effects (font (size 1.27 1.27)) hide)
@@
     (in_bom yes) (on_board yes) (fields_autoplaced)
     (property "Reference" "R2" (id 0) (at 111.76 62.5942 90))
-    (property "Value" "" (id 1) (at 111.76 65.1311 90))
+    (property "Value" "92R" (id 1) (at 111.76 65.1311 90))
     (property "Footprint" "" (id 2) (at 111.76 69.088 90)
       (effects (font (size 1.27 1.27)) hide)
@@
       (effects (font (size 1.27 1.27)) (justify left))
     )
-    (property "Value" "" (id 1) (at 170.053 77.9022 90)
-      (effects (font (size 1.27 1.27)) (justify left))
-    )
+    (property "Value" "SW_SPST" (id 1) (at 170.053 77.9022 90)
+      (effects (font (size 1.27 1.27)) (justify left))
+    )
